File: hardware/stm32-netnode.kicad_sch (KiCad schematic)
At the start: 96 parts, among them J1 USB4110-GF-A, J2 J0011D01BNL, J4 Breakout, SW1 7914J-1-000E, SW2 7914J-1-000E, U1 STM32F407VETx, U2 W25Q25PWSSIQ, U3 LAN8720A, U4 BME688, U5 CP2102N-A02-GQFN20R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

Commit message: Radd rev 2.0
Parts:
- removed C3: 0.1u, Capacitor_SMD:C_0603_1608Metric, symbol Device:C_Small
- removed C4: 4.7u, Capacitor_SMD:C_0805_2012Metric, symbol Device:C_Small
- removed D1, D2: LED, LED_SMD:LED_0603_1608Metric, symbol Device:LED
- removed H1, H2, H3, H4: MountingHole_Pad, MountingHole:MountingHole_2.7mm_M2.5_Pad_Via, symbol Mechanical:MountingHole_Pad
- removed J4: Breakout, Connector_PinHeader_2.54mm:PinHeader_2x10_P2.54mm_Vertical_SMD, symbol Connector_Generic:Conn_02x10_Odd_Even
- removed R28: 1k, Resistor_SMD:R_0603_1608Metric, symbol Device:R_Small
- removed R3, R4: 4.7k, Resistor_SMD:R_0603_1608Metric, symbol Device:R_Small
- removed R31, R32: 220, Resistor_SMD:R_0603_1608Metric, symbol Device:R_Small
- removed SW1, SW2: 7914J-1-000E, footprints:SW_7914J-1-000E, symbol Switch:SW_Push
- removed TP5, TP6: TestPoint, TestPoint:TestPoint_Pad_D1.5mm, symbol Connector:TestPoint
- removed U5: CP2102N-A02-GQFN20R, footprints:SILABS_CP2102N-A02-GQFN20R, symbol CP2102N-A02-GQFN20R:CP2102N-A02-GQFN20R
- added D1: WS2812B, LED_SMD:LED_WS2812B_PLCC4_5.0x5.0mm_P3.2mm, symbol LED:WS2812B
- added J3: UART5, Connector_PinHeader_2.54mm:PinHeader_1x03_P2.54mm_Vertical, symbol Connector_Generic:Conn_01x03
- added J4: SWD, Connector_PinHeader_2.54mm:PinHeader_1x04_P2.54mm_Vertical, symbol Connector_Generic:Conn_01x04
- added J5: I2C, footprints:CONN4_BM04B-SRSS_JST, symbol Connector_Generic:Conn_01x04
- added J6: SPI2, footprints:CONN_BM06B-SRSS-TB_JST, symbol Connector_Generic:Conn_01x06
- added SW3: BOOT0, footprints:SW_7914J-1-000E, symbol Switch:SW_Push_Open_Dual
- added SW4: NRST, footprints:SW_7914J-1-000E, symbol Switch:SW_Push_Open_Dual
- C1: value 10u -> 100nF
- C2: value 10u -> 4.7u
- C21, C22: value 27pF -> 12pF; footprint Capacitor_SMD:C_0603_1608Metric -> Capacitor_SMD:C_0402_1005Metric
- C28: value 10u -> 4.7u; footprint Capacitor_SMD:C_0603_1608Metric -> Capacitor_SMD:C_0805_2012Metric
- FB1: footprint Inductor_SMD:L_0201_0603Metric -> Inductor_SMD:L_0603_1608Metric
- R27: value 10k -> 0
- U2: value W25Q25PWSSIQ -> W25Q80DVUXIE TR
- Y2: value ABM3B-25.000MHZ-B2-T -> ECS-250-8-30B-CKM; footprint Crystal:Crystal_SMD_Abracon_ABM3B-4Pin_5.0x3.2mm -> footprints:XTAL_ECS-250-8-30B-CKM
Connections:
- net VDDIO is gone; now on net +3.3V: C16.1, R15.1, R16.1, R17.1, R18.1, U3.9 (VDDIO)
- net +3.3V: now also D1.1 (VDD), J5.2 (Pin_2), J6.2 (Pin_2), SW3.1
- net BOOT0: now also SW3.4
- net FLASH_CE: now also U1.88 (PD7); no longer U1.35 (PB0)
- net GND: now also J2.8 (GND), D1.3 (VSS), J3.3 (Pin_3), J4.1 (Pin_1), J5.1 (Pin_1), J6.1 (Pin_1), SW4.3
- net I2C3_SCL: now also J5.4 (Pin_4)
- net I2C3_SDA: now also J5.3 (Pin_3)
- net NRST: now also J4.4 (Pin_4), SW4.2
- net SPI2_CS: now also J6.6 (Pin_6); no longer U1.3 (PE4)
- net SPI2_MISO: now also J6.5 (Pin_5)
- net SPI2_MOSI: now also J6.4 (Pin_4)
- net SPI2_SCK: now also J6.3 (Pin_3)
- net UART5_RX: now also U1.83 (PD2), J3.1 (Pin_1); no longer U1.82 (PD1)
- net UART5_TX: now also J3.2 (Pin_2)
- net USB_D+: now also U1.71 (PA12)
- net USB_D-: now also U1.70 (PA11)
- net NEOPIX: now reaches U1.46 (PE15)
- net NEOPIX: now also D1.4 (DIN)
- net SWDIO: now reaches U1.72 (PA13)
- net SWDIO: now also J4.3 (Pin_3)
- net SWCLK: now reaches U1.76 (PA14)
- net SWCLK: now also J4.2 (Pin_2)
- net ADC1_IN0: no longer names the net of U1.23 (PA0)
- net ADC1_IN3: no longer names the net of U1.26 (PA3)
- net DAC1_OUT: no longer names the net of U1.29 (PA4)
- net GPIO1: no longer names the net of U1.1 (PE2)
- net PWM_TIM4_CH3: no longer names the net of U1.95 (PB8)
- net PWM_TIM4_CH4: no longer names the net of U1.96 (PB9)
- net UART4_RX: no longer names the net of U1.79 (PC11)
- net UART4_TX: no longer names the net of U1.78 (PC10)
- no-connect marks 7 -> 2
Other:
- note added: "Add option to limit rise time on clock line with 0ohm"
- note added: "ETHERNET"
- note added: "Flash/Temp"
- note added: "Headers"
- note added: "MCU"
- note added: "STM32 NETNODE Rev 2.0"
- note added: "USB/Power"
- title: (none) -> STM32 Netnode
- moved on the sheet: C1, C10, C11, C12, C13, C14, C15, C16, C17, C18, C19, C2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
